Commit message: Patch Aloha.urdf joint limits: real SO-101 values for arms, placeholder for lift
Arm joints (left/right_joint1..6) now carry the real limits read off
SO-ARM101-USD.usd (converted deg->rad) plus effort=30/velocity=3.0 matching
NVIDIA's tuned simulation values. vertical_move (lift) gets a placeholder
0-0.3m range -- no authoritative spec found, flagged for empirical correction
once the mesh is visually inspected in Phase 2.

Verified: URDF still parses (18 joints, 19 links, unchanged), zero remaining
zeroed-limit blocks. Polarity (sign of each range) not yet verified against
this URDF's own axis vectors -- noted in CLAUDE.md as a Phase 2 check.

Co-Authored-By: Claude Sonnet 5 <noreply@anthropic.com>

File: assets/upstream_alohamini1/urdf/Aloha.urdf (robot description, URDF)
Before this commit: robot Aloha, 19 links, 18 joints
Joints:
- joint left_joint1: limit lower=0 upper=0 effort=0 velocity=0 -> lower=-1.919860 upper=1.919860 effort=30 velocity=3.0
- joint left_joint2: limit lower=0 upper=0 effort=0 velocity=0 -> lower=-1.745330 upper=1.745330 effort=30 velocity=3.0
- joint left_joint3: limit lower=0 upper=0 effort=0 velocity=0 -> lower=-1.745330 upper=1.570800 effort=30 velocity=3.0
- joint left_joint4: limit lower=0 upper=0 effort=0 velocity=0 -> lower=-1.658060 upper=1.658060 effort=30 velocity=3.0
- joint left_joint5: limit lower=0 upper=0 effort=0 velocity=0 -> lower=-2.792530 upper=2.792530 effort=30 velocity=3.0
- joint left_joint6: limit lower=0 upper=0 effort=0 velocity=0 -> lower=-0.174533 upper=1.745330 effort=30 velocity=3.0
- joint right_joint1: limit lower=0 upper=0 effort=0 velocity=0 -> lower=-1.919860 upper=1.919860 effort=30 velocity=3.0
- joint right_joint2: limit lower=0 upper=0 effort=0 velocity=0 -> lower=-1.745330 upper=1.745330 effort=30 velocity=3.0
- joint right_joint3: limit lower=0 upper=0 effort=0 velocity=0 -> lower=-1.745330 upper=1.570800 effort=30 velocity=3.0
- joint right_joint4: limit lower=0 upper=0 effort=0 velocity=0 -> lower=-1.658060 upper=1.658060 effort=30 velocity=3.0
- joint right_joint5: limit lower=0 upper=0 effort=0 velocity=0 -> lower=-2.792530 upper=2.792530 effort=30 velocity=3.0
- joint right_joint6: limit lower=0 upper=0 effort=0 velocity=0 -> lower=-0.174533 upper=1.745330 effort=30 velocity=3.0
- joint vertical_move: limit lower=0 upper=0 effort=0 velocity=0 -> lower=0.000000 upper=0.300000 effort=200 velocity=0.1

Commit message: Fix lift travel range with real spec; add verified LeKiwi wheel kinematics
Corrected vertical_move upper limit from a 0.3m guess to the real 0.6m spec
(liyiteng/lerobot_alohamini's lift_axis.py: soft_max_mm=600, lead screw
84mm/rev -- matches alohamini1's model_specs.py exactly).

Added scripts/alohamini1_specs.py as a single source of truth for constants
used across scripts: arm joint gains, lift range, and LeKiwi holonomic wheel
kinematics (wheel_radius=0.05m, base_radius=0.125m, verified against the exact
raw source, not a paraphrase). Caught and fixed a real mapping bug in the
process: our URDF's wheel1/wheel2/wheel3 do NOT naively align with the
reference code's wheel-angle order -- verified by computing each wheel's
actual position angle from its URDF joint origin (wheel1~149deg,
wheel3~-91deg, wheel2~30deg), giving the correct pairing
["wheel1","wheel3","wheel2"] against angles [150,-90,30].

Co-Authored-By: Claude Sonnet 5 <noreply@anthropic.com>

File: assets/upstream_alohamini1/urdf/Aloha.urdf (robot description, URDF)
Before this commit: robot Aloha, 19 links, 18 joints
Joints:
- joint vertical_move: limit lower=0.000000 upper=0.300000 effort=200 velocity=0.1 -> lower=0.000000 upper=0.600000 effort=200 velocity=0.15

Commit message: Fix gripper not fully closing: real joint limit didn't match this mesh
NVIDIA's SO-ARM101-USD.usd reference gives real, correctly-read Jaw limits
(-0.174533 to 1.745329 rad), but they don't transfer to AlohaMini1's own STL
mesh -- different CAD source, different jaw linkage geometry, despite being
nominally "the same" SO-101 arm design. User reported the gripper wasn't
closing all the way; confirmed empirically rather than guessing: widened the
limit temporarily, swept several joint angles, rendered close-up screenshots
at each. -0.174533 leaves a visible gap (not closed), 1.745329 is genuinely
fully open, and the fingers actually meet at -1.570796 (-90 degrees) -- well
outside the original range entirely.

Corrected the real limit in Aloha.urdf for both left_joint6 and right_joint6
(not just a script-side clamp), updated JAW_OPEN_RAD/JAW_CLOSED_RAD and
ARM_JOINT_LIMITS_RAD[6] in alohamini1_specs.py to match, and reran the full
pipeline (reimport -> rebuild scene -> reconfigure physics -> refix wheel
collision). Reverified: docs/gripper_closed_final.png shows the fingers
actually touching, and verify_physics.py still passes with the wider range
(no NaN/Inf, exact convergence, stable base height).

Co-Authored-By: Claude Sonnet 5 <noreply@anthropic.com>

File: assets/upstream_alohamini1/urdf/Aloha.urdf (robot description, URDF)
Before this commit: robot Aloha, 19 links, 18 joints
Joints:
- joint left_joint6: limit lower=-0.174533 upper=1.745330 effort=30 velocity=3.0 -> lower=-1.570796 upper=1.745330 effort=30 velocity=3.0
- joint right_joint6: limit lower=-0.174533 upper=1.745330 effort=30 velocity=3.0 -> lower=-1.570796 upper=1.745330 effort=30 velocity=3.0

Commit message: Widen gripper close margin, verify self-collision works, add lift joystick control
1. Widened gripper close limit further per request (-1.570796 -> -1.85 rad,
   ~-106 deg) for more squeeze margin gripping thin objects. Verified visually
   clean at -1.85 and -2.0 (no bad mesh interpenetration); settled on -1.85.

2. Verified arm-to-arm self-collision is actually working, not just "doesn't
   destabilize rest pose" (which was all that was verified before). Direct
   test: drove both arms' joint1 toward each other -- they got physically
   stuck partway (commanded -1.9 rad, only reached 0.66 rad) with heavily
   overlapping wrist-link bounding boxes, confirming a real collision stopped
   the motion. docs/self_collision_verified.png shows the two gripper
   end-effectors properly in contact. (First attempt used the wrong rotation
   sign and showed the arms moving apart, which looked like nothing was
   happening -- real lesson: verify the test itself actually brings parts
   together before concluding collision "isn't working".)

3. Added lift control to the joystick scheme: Triangle=up, Square=down, same
   increment-while-held pattern as the gripper, independent of L1/L2/R2 mode
   selection so it works no matter what's currently selected. Verified the
   underlying increment/clamp logic directly (0 -> 0.065 -> 0.14 -> 0.215m
   over 1.5s, matching the expected rate). On joystick_bridge_local.py (the
   macOS/pygame side actually in use), button indices 2/3 for square/triangle
   are inferred from standard SDL face-button ordering, not individually
   confirmed one-at-a-time like L1/R1 were -- verify with --debug if it
   doesn't respond as expected.

Reran the full pipeline (reimport -> rebuild scene -> reconfigure physics ->
refix wheel collision) for the gripper limit change and reverified overall
stability (verify_physics.py: no NaN/Inf, exact convergence, stable base
height).

Co-Authored-By: Claude Sonnet 5 <noreply@anthropic.com>

File: assets/upstream_alohamini1/urdf/Aloha.urdf (robot description, URDF)
Before this commit: robot Aloha, 19 links, 18 joints
Joints:
- joint left_joint6: limit lower=-1.570796 upper=1.745330 effort=30 velocity=3.0 -> lower=-1.850000 upper=1.745330 effort=30 velocity=3.0
- joint right_joint6: limit lower=-1.570796 upper=1.745330 effort=30 velocity=3.0 -> lower=-1.850000 upper=1.745330 effort=30 velocity=3.0
